File: schematic/Wireless_eBike_V1.sch (KiCad schematic (older format))
At the start: 16 parts

Commit message: Updated schematic
Parts:
- added U?: nRF52840_Blue_Dongle, symbol Wireless_eBike-cache:nRF52840_Blue_Dongle
- D? (x2): symbol D_Schottky -> Device:D_Schottky
- F? (x2): symbol FUSE -> Device:Fuse
- K?: symbol 6-Way_Higo -> Dongle:6-Way_Higo
- K?: symbol 8-Way_Higo -> Dongle:8-Way_Higo
- P?: symbol CONN_01X04 -> Wireless_eBike-cache:CONN_01X04
- P? (x4): symbol CONN_01X03 -> Wireless_eBike-cache:CONN_01X03
- R? (x2): symbol R -> Device:R
- U?: symbol BTS4140N -> Wireless_eBike-cache:BTS4140N
- U?: value nRF52840 -> nRF52840 MDK Dongle; symbol nRF52840 -> Wireless_eBike-cache:nRF52840_MDK_Dongle
- U?: symbol Generic_DC-DC -> Wireless_eBike-cache:Generic_DC-DC
Connections:
- net GND: now also U?.3 (OUT-), U?.8 (P21), U?.3 (GND)
- net Red: now also F?.2; no longer F?.1
- net SWDCLK: now also U?.11 (DIO)
- net SWDIO: now also U?.11 (DIO)
- net TSDZ2_5V_Output: now also F?.1; no longer F?.2
- net MotorON: now reaches U?.1 (IN), U?.6 (P5)
- net MotorON: now also U?.4 (1.00)
- net RX: now reaches R?.1, U?.4 (P7)
- net RX: now also U?.5 (0.29)
- net TX: now reaches R?.1, U?.5 (P6)
- net TX: now also U?.6 (0.22)
- net 5V: now reaches U?.9 (P2)
- net 5V: now also F?.1, U?.1 (VBUS)
- net at F?.2: now also U?.4 (OUT+); no longer U?.9 (P2)
Other:
- note added: "Only one nRF52840 Board is required, \nmake sure to follow the pin layout of \nwhichever one you have"
Changed lines of the file:
@@
-EESchema Schematic File Version 2
-LIBS:power
-LIBS:device
-LIBS:transistors
-LIBS:conn
-LIBS:linear
-LIBS:regul
-LIBS:74xx
-LIBS:cmos4000
-LIBS:adc-dac
-LIBS:memory
-LIBS:xilinx
-LIBS:microcontrollers
-LIBS:dsp
-LIBS:microchip
-LIBS:analog_switches
-LIBS:motorola
-LIBS:texas
-LIBS:intel
-LIBS:audio
-LIBS:interface
-LIBS:digital-audio
-LIBS:philips
-LIBS:display
-LIBS:cypress
-LIBS:siliconi
-LIBS:opto
-LIBS:atmel
-LIBS:contrib
-LIBS:valves
-LIBS:Dongle
-LIBS:Wireless_eBike_V1-cache
-EELAYER 25 0
+EESchema Schematic File Version 4
+EELAYER 30 0
 EELAYER END
 $Descr A4 11693 8268
@@
 $EndDescr
 $Comp
-L BTS4140N U?
+L Wireless_eBike-cache:BTS4140N U?
 U 1 1 5EEB0A4F
 P 9250 2050
@@
 $EndComp
 $Comp
-L nRF52840 U?
-U 1 1 5EEB15B7
-P 7750 3400
-F 0 "U?" H 7750 3450 60  0000 C CNN
-F 1 "nRF52840" H 7750 2850 60  0000 C CNN
-F 2 "" H 7750 3400 60  0000 C CNN
-F 3 "" H 7750 3400 60  0000 C CNN
-	1    7750 3400
-	1    0    0    -1
-$EndComp
-$Comp
-L CONN_01X04 P?
+L Wireless_eBike-cache:CONN_01X04 P?
 U 1 1 5EEB15DE
 P 10300 3150
@@
 $EndComp
 $Comp
-L Generic_DC-DC U?
+L Wireless_eBike-cache:Generic_DC-DC U?
 U 1 1 5EEB1756
 P 5600 2400
@@
 NoConn ~ 8300 2900
 $Comp
-L 6-Way_Higo K?
+L Dongle:6-Way_Higo K?
 U 1 1 5EEB225F
 P 2350 3500
@@
 $EndComp
 $Comp
-L 8-Way_Higo K?
+L Dongle:8-Way_Higo K?
 U 1 1 5EEB22D5
 P 2300 2100
@@
 NOTE - The brake input to the TSDZ2 is pulled up to 5V\nby a resistor inside the motor controller. Pull the input\nto GND to activate. This is normally done with a switch\n(2-Pin Connector). If you have the 8-Way Higo cable\nyou can use a via a powered brake sensor with 3-wires.
 $Comp
-L CONN_01X03 P?
+L Wireless_eBike-cache:CONN_01X03 P?
 U 1 1 5EEB45E0
 P 2000 6200
@@
 $EndComp
 $Comp
-L CONN_01X03 P?
+L Wireless_eBike-cache:CONN_01X03 P?
 U 1 1 5EEB4667
 P 2000 6800
@@
 	9350 2500 9900 2500
 Wire Wire Line
-	5000 1650 9250 1650
-Wire Wire Line
-	8300 3000 10100 3000
-Wire Wire Line
-	8300 3100 10100 3100
-Wire Wire Line
-	8300 3200 10100 3200
-Wire Wire Line
-	8300 3300 10100 3300
-Wire Wire Line
-	6100 2300 6250 2300
+	5000 1650 8850 1650
 Wire Wire Line
 	2900 3100 3200 3100
@@
 	4900 2500 5100 2500
 Wire Wire Line
-	4900 2300 5100 2300
+	4900 2300 5000 2300
 Connection ~ 8850 1650
 Connection ~ 5000 2300
 Wire Wire Line
-	8300 3400 9150 3400
-Wire Wire Line
 	2200 5050 2650 5050
 Wire Wire Line
 	2650 5050 2650 4550
 Wire Wire Line
-	2200 4550 3350 4550
+	2200 4550 2650 4550
 Wire Wire Line
 	2200 4650 2550 4650
@@
 	2550 4650 2550 5150
 Wire Wire Line
-	2200 5150 2900 5150
+	2200 5150 2550 5150
 Connection ~ 2650 4550
 Connection ~ 2550 5150
@@
 	2500 6300 2500 6900
 Wire Wire Line
-	2200 6900 2850 6900
+	2200 6900 2500 6900
 Wire Wire Line
 	2200 6200 2600 6200
 Wire Wire Line
-	2600 6200 2600 6800
+	2600 6200 2600 6500
 Wire Wire Line
 	2600 6800 2200 6800
 Wire Wire Line
-	2200 6100 3300 6100
+	2200 6100 2700 6100
 Wire Wire Line
 	2700 6100 2700 6700
@@
 	3300 6900 3150 6900
 $Comp
-L D_Schottky D?
+L Device:D_Schottky D?
 U 1 1 5EEBA014
 P 3050 5150
@@
 F 1 "D_Schottky" H 3050 5050 50  0000 C CNN
 F 2 "" H 3050 5150 50  0000 C CNN
-F 3 "" H 3050 5150 50  0000 C CNN
+F 3 "~" H 3050 5150 50  0000 C CNN
 	1    3050 5150
 	1    0    0    -1
 $EndComp
 $Comp
-L D_Schottky D?
+L Device:D_Schottky D?
 U 1 1 5EEBA05E
 P 3000 6900
@@
 Yellow
 $Comp
-L FUSE F?
-U 1 1 5EEBC0DD
-P 3000 6500
-F 0 "F?" H 3100 6550 50  0000 C CNN
-F 1 "PTC_FUSE" H 3000 6400 50  0000 C CNN
-F 2 "" H 3000 6500 50  0000 C CNN
-F 3 "" H 3000 6500 50  0000 C CNN
-	1    3000 6500
-	1    0    0    -1
-$EndComp
-$Comp
-L R R?
+L Device:R R?
 U 1 1 5EEBCDCD
 P 5900 3500
@@
 F 1 "2K" V 5900 3500 50  0000 C CNN
 F 2 "" V 5830 3500 50  0000 C CNN
-F 3 "" H 5900 3500 50  0000 C CNN
+F 3 "~" H 5900 3500 50  0000 C CNN
 	1    5900 3500
 	0    1    1    0
 $EndComp
-Wire Wire Line
-	7200 3500 6050 3500
 Wire Wire Line
 	5750 3500 4900 3500
 Text Notes 5200 4100 0    60   ~ 0
 Current-limiting 2K resistor to allow\n5V TSDZ2 UART Tx to work with the\n3.3V nRF52840 UART Rx. Going in\nthe other direction is okay because\n3.3V is considered HIGH in 5V logic.
-Wire Wire Line
-	3300 6500 3250 6500
-Wire Wire Line
-	2750 6500 2600 6500
 Text Notes 1600 7500 0    60   ~ 0
 Diode to protect from high voltage into brake input, use\na Schottky type to reduce the dropped voltage when it's\nconducting. The Fuse is a PPTC self-resetting type to\nprotect the TSDZ2 5V - 50mA should be about right.
-$Comp
-L FUSE F?
-U 1 1 5EEBDA76
-P 6500 2300
-F 0 "F?" H 6600 2350 50  0000 C CNN
-F 1 "PTC_FUSE" H 6400 2200 50  0000 C CNN
-F 2 "" H 6500 2300 50  0000 C CNN
-F 3 "" H 6500 2300 50  0000 C CNN
-	1    6500 2300
-	1    0    0    -1
-$EndComp
-Wire Wire Line
-	7200 3000 7000 3000
-Wire Wire Line
-	7000 3000 7000 2300
-Wire Wire Line
-	7000 2300 6750 2300
 Wire Notes Line
 	2800 5300 2800 5000
@@
 Optional fuse, value around 250mA,\ndepends on hardware and firmware.
 $Comp
-L R R?
+L Device:R R?
 U 1 1 5EF0E0CE
 P 5900 3400
@@
 F 1 "100R" V 5900 3400 50  0000 C CNN
 F 2 "" V 5830 3400 50  0000 C CNN
-F 3 "" H 5900 3400 50  0000 C CNN
+F 3 "~" H 5900 3400 50  0000 C CNN
 	1    5900 3400
 	0    1    -1   0
 $EndComp
 Wire Wire Line
-	7200 3400 6050 3400
-Wire Wire Line
 	5750 3400 4900 3400
 Wire Wire Line
 	5000 2300 5000 1650
-Wire Wire Line
-	7200 3100 6500 3100
 Wire Wire Line
 	6500 3100 6500 2500
@@
 2-WIRE BRAKE\n  SWITCHES
 $Comp
-L CONN_01X03 P?
+L Wireless_eBike-cache:CONN_01X03 P?
 U 1 1 5EF1F31E
 P 2000 4650
@@
 $EndComp
 $Comp
-L CONN_01X03 P?
+L Wireless_eBike-cache:CONN_01X03 P?
 U 1 1 5EF1F377
 P 2000 5150
@@
 NoConn ~ 2200 5250
 NoConn ~ 3800 8100
+Wire Wire Line
+	8850 1650 9250 1650
+Wire Wire Line
+	5000 2300 5100 2300
+Wire Wire Line
+	2650 4550 3350 4550
+Wire Wire Line
+	2550 5150 2900 5150
+Wire Wire Line
+	2700 6100 3300 6100
+Wire Wire Line
+	2600 6500 2600 6800
+Wire Wire Line
+	2500 6900 2850 6900
+Text GLabel 7130 3400 0    50   Input ~ 0
+TX
+Text GLabel 7140 3500 0    50   Input ~ 0
+RX
+Text GLabel 7140 3000 0    50   Input ~ 0
+5V
+Text GLabel 7200 3100 0    50   Input ~ 0
+GND
+Wire Wire Line
+	6500 3100 6750 3100
+Wire Wire Line
+	7000 2300 7000 2900
+Text GLabel 8300 3400 2    50   Input ~ 0
+MotorON
+Text GLabel 9050 3400 0    50   Input ~ 0
+MotorON
+Wire Wire Line
+	9050 3400 9150 3400
+Text GLabel 6750 3100 2    50   Input ~ 0
+GND
+Wire Wire Line
+	6700 2900 6700 3000
+Wire Wire Line
+	7000 2900 6700 2900
+Text GLabel 6810 3000 2    50   Input ~ 0
+5V
+Text GLabel 6810 3500 2    50   Input ~ 0
+RX
+Text GLabel 6820 3400 2    50   Input ~ 0
+TX
+Wire Wire Line
+	7140 3000 7200 3000
+Wire Wire Line
+	6700 3000 6810 3000
+Wire Wire Line
+	7130 3400 7200 3400
+Wire Wire Line
+	7200 3500 7140 3500
+Wire Wire Line
+	6050 3500 6810 3500
+Wire Wire Line
+	6820 3400 6050 3400
+Text GLabel 8450 3000 2    50   Input ~ 0
+GND
+Text GLabel 8380 3300 2    50   Input ~ 0
+SWDIO
+Text GLabel 8310 3200 2    50   Input ~ 0
+SWDCLK
+Text GLabel 8470 3100 2    50   Input ~ 0
+RST
+Wire Wire Line
+	8300 3200 8310 3200
+Wire Wire Line
+	8300 3300 8380 3300
+Wire Wire Line
+	8300 3100 8470 3100
+Wire Wire Line
+	8300 3000 8450 3000
+Text GLabel 8970 3300 0    50   Input ~ 0
+SWDIO
+Text GLabel 9030 3200 0    50   Input ~ 0
+SWDCLK
+Text GLabel 8870 3100 0    50   Input ~ 0
+RST
+Text GLabel 8890 3000 0    50   Input ~ 0
+GND
+Wire Wire Line
+	10100 3000 8890 3000
+Wire Wire Line
+	10100 3100 8870 3100
+Wire Wire Line
+	10100 3200 9030 3200
+Wire Wire Line
+	10100 3300 8970 3300
+$Comp
+L Device:Fuse F?
+U 1 1 5EEBC0DD
+P 3000 6500
+F 0 "F?" H 3100 6550 50  0000 C CNN
+F 1 "PTC_FUSE" H 3000 6400 50  0000 C CNN
+F 2 "" H 3000 6500 50  0000 C CNN
+F 3 "" H 3000 6500 50  0000 C CNN
+	1    3000 6500
+	0    1    1    0
+$EndComp
+$Comp
+L Wireless_eBike-cache:nRF52840_MDK_Dongle U?
+U 1 1 5EEB15B7
+P 7750 3400
+F 0 "U?" H 7750 3450 60  0000 C CNN
+F 1 "nRF52840 MDK Dongle" H 7750 2850 60  0000 C CNN
+F 2 "" H 7750 3400 60  0000 C CNN
+F 3 "" H 7750 3400 60  0000 C CNN
+	1    7750 3400
+	1    0    0    -1
+$EndComp
+$Comp
+L Device:Fuse F?
+U 1 1 5EEBDA76
+P 6500 2300
+F 0 "F?" H 6600 2350 50  0000 C CNN
+F 1 "PTC_FUSE" H 6400 2200 50  0000 C CNN
+F 2 "" H 6500 2300 50  0000 C CNN
+F 3 "" H 6500 2300 50  0000 C CNN
+	1    6500 2300
+	0    1    1    0
+$EndComp
+$Comp
+L Wireless_eBike-cache:nRF52840_Blue_Dongle U?
+U 1 1 5F10C6B5
+P 8300 5670
+F 0 "U?" H 8240 5740 60  0000 C CNN
+F 1 "nRF52840_Blue_Dongle" H 8280 5090 60  0000 C CNN
+F 2 "" H 8300 5670 60  0000 C CNN
+F 3 "" H 8300 5670 60  0000 C CNN
+	1    8300 5670
+	1    0    0    -1
+$EndComp
+Text GLabel 8900 5070 2    50   Input ~ 0
+SWDCLK
+Wire Wire Line
+	8750 5070 8900 5070
+Text GLabel 7590 5070 0    50   Input ~ 0
+SWDIO
+Text GLabel 8910 5370 2    50   Input ~ 0
+GND
+Text GLabel 8900 5170 2    50   Input ~ 0
+5V
+Text GLabel 7590 5770 0    50   Input ~ 0
+MotorON
+Text GLabel 7580 5570 0    50   Input ~ 0
+TX
+Text GLabel 7590 5670 0    50   Input ~ 0
+RX
+Wire Wire Line
+	8850 5170 8900 5170
+Wire Wire Line
+	8850 5370 8910 5370
+Wire Wire Line
+	7750 5070 7590 5070
+Wire Wire Line
+	7590 5670 7650 5670
+Wire Wire Line
+	7580 5570 7650 5570
+Wire Wire Line
+	7650 5770 7590 5770
+Wire Notes Line
+	7000 4650 10300 4650
+Wire Notes Line
+	10300 4650 10300 6450
+Wire Notes Line
+	10300 6450 7000 6450
+Wire Notes Line
+	7000 6450 7000 4650
+Text Notes 8750 4950 0    50   ~ 0
+Only one nRF52840 Board is required, \nmake sure to follow the pin layout of \nwhichever one you have
+Wire Wire Line
+	6650 2300 7000 2300
+Wire Wire Line
+	6100 2300 6350 2300
+Wire Wire Line
+	2600 6500 2850 6500
+Wire Wire Line
+	3150 6500 3300 6500
 $EndSCHEMATC
