File: EBike_wireless_TSDZ2/schematic/wired_remote/Wired_remote.sch (KiCad schematic (older format))
At the start: 12 parts

Commit message: Updated the wired remote page, to export a PNG image without showing the details of page author, etc
Parts:
- U?: symbol Wireless_Ebike:BSP296 -> Wired_remote-rescue:BSP296-Wireless_Ebike
- U?: symbol Wireless_Ebike:BTS4140N-Wireless_eBike -> Wired_remote-rescue:BTS4140N-Wireless_eBike-Wireless_Ebike
- U?: symbol Wireless_Ebike:Generic_DC-DC-Wireless_eBike -> Wired_remote-rescue:Generic_DC-DC-Wireless_eBike-Wireless_Ebike
Other:
- moved on the sheet: Brake, button_1, button_2, button_3, button_4
